Commit message: Upload f1tenth model

File: F110.export.urdf (robot description, URDF)
Before this commit: robot racecar, 13 links, 12 joints
Links:
- link chassis: geometry visual mesh filename=x:\F1tenth-Genesis\f1tenth_model\meshes\chassis.STL
- link laser: geometry collision box size=0.1 0.1 0.1; visual mesh filename=x:\F1tenth-Genesis\f1tenth_model\meshes\hokuyo.dae
- link left_front_wheel: geometry collision cylinder length=0.045 radius=0.05; visual mesh filename=x:\F1tenth-Genesis\f1tenth_model\meshes\left_front_wheel.STL
- link left_rear_wheel: geometry collision cylinder length=0.045 radius=0.05; visual mesh filename=x:\F1tenth-Genesis\f1tenth_model\meshes\left_rear_wheel.STL
- link left_steering_hinge: geometry visual mesh filename=x:\F1tenth-Genesis\f1tenth_model\meshes\left_steering_hinge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
- link right_front_wheel: geometry collision cylinder length=0.045 radius=0.05; visual mesh filename=x:\F1tenth-Genesis\f1tenth_model\meshes\right_front_wheel.S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
- link right_rear_wheel: geometry collision cylinder length=0.045 radius=0.05; visual mesh filename=x:\F1tenth-Genesis\f1tenth_model\meshes\right_rear_wheel.STL
- link right_steering_hinge: geometry visual mesh filename=x:\F1tenth-Genesis\f1tenth_model/meshes/right_steering_hing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

Commit message: Local work before linking remote

File: F110.export.urdf (robot description, URDF)
Before this commit: robot racecar, 13 links, 12 joints
Links:
- link chassis: geometry visual mesh filename=f1tenth_model/meshes/chassis.STL
- link laser: geometry collision box size=0.1 0.1 0.1; visual mesh filename=f1tenth_model/meshes/hokuyo.dae
- link left_front_wheel: geometry collision cylinder length=0.045 radius=0.05; visual mesh filename=f1tenth_model/meshes/left_front_wheel.STL
- link left_rear_wheel: geometry collision cylinder length=0.045 radius=0.05; visual mesh filename=f1tenth_model/meshes/left_rear_wheel.STL
- link left_steering_hinge: geometry visual mesh filename=f1tenth_model/meshes/left_steering_hinge.STL
- link right_front_wheel: geometry collision cylinder length=0.045 radius=0.05; visual mesh filename=f1tenth_model/meshes/right_front_wheel.STL
- link right_rear_wheel: geometry collision cylinder length=0.045 radius=0.05; visual mesh filename=f1tenth_model/meshes/right_rear_wheel.STL
- link right_steering_hinge: geometry visual mesh filename=f1tenth_model/meshes/right_steering_hinge.STL
