Commit message: Add standalone QRSAC trainer and force-based vehicle physics.
Single-process training without Reverb/Redis, updated env drive/aero model and URDF params, plus bench/diagnostic scripts for physics validation.

Co-authored-by: Cursor <cursoragent@cursor.com>

File: F110.export.urdf (robot description, URDF)
Before this commit: robot racecar, 13 links, 12 joints
Links:
- link chassis_inertia: mass 4.0 -> 2.05
Joints:
- joint left_steering_hinge_joint: limit lower=-1.0 upper=1.0 effort=10 velocity=100 -> lower=-0.44 upper=0.44 effort=10 velocity=100
- joint right_steering_hinge_joint: limit lower=-1.0 upper=1.0 effort=10 velocity=100 -> lower=-0.44 upper=0.44 effort=10 velocity=100
